Commit message: Added first layer to omni robot and lidar scanner

File: src/omni_robot/xacro/lidar.urdf.xacro (robot description, xacro)
@@ -7,5 +7,5 @@
             <origin xyz="0 0 0" rpy="0 0 0"/>
             <geometry>
-            <box size="0.1 0.1 0.1"/>
+            <box size="${scale*0.1} ${scale*0.1} ${scale*0.1}"/>
             </geometry>
             </collision>

File: src/omni_robot/xacro/main.urdf.xacro (robot description, xacro)
@@ -1,5 +1,5 @@
 <?xml version="1.0"?>
 <robot xmlns:xacro="http://www.ros.org/wiki/xacro" name="omni_robot">
-		<!-- Gazebo plugins -->
+	<!-- Gazebo plugins -->
 	<xacro:include filename="$(find omni_robot)/gazebo/omni_robot.gazebo" />
 	<!-- Robot components -->
@@ -64,5 +64,5 @@
 	/>
 	<xacro:lidar_macro
-		xyz="0 0 0.03"
+		xyz="0 0 0.04"
 		rpy="0 0 0"
 		scale = "0.3"
